Commit message: starting with hardware interface

File: description/ros2_control.xacro (robot description, xacro)
@@ -1,5 +1,5 @@
 <?xml version="1.0"?>
 <robot xmlns:xacro="http://www.ros.org/wiki/xacro">
-<ros2_control name="GazeboSystem" type="system">
+<!-- <ros2_control name="GazeboSystem" type="system">
     <hardware>
         <plugin>gazebo_ros2_control/GazeboSystem</plugin>
@@ -21,4 +21,34 @@
         <state_interface name="position" />
     </joint>
+</ros2_control> -->
+<!-- TODO: toggle -->
+<ros2_control name="RealRobot" type="system">
+    <hardware>
+        <plugin>diffdrive_arduino/DiffDriveArduino</plugin>
+        <param name="left_wheel_name">left_wheel_joint</param>
+        <param name="right_wheel_name">right_wheel_joint</param>
+        <param name="loop_rate">30</param>
+        <param name="device">/dev/ttyUSB0</param>
+        <param name="baud_rate">57600</param>
+        <param name="timeout">1000</param>
+        <param name="enc_counts_per_rev">3436</param>
+    </hardware>
+    <!-- Note everything below here is the same as the Gazebo one -->
+    <joint name="left_wheel_joint">
+        <command_interface name="velocity">
+            <param name="min">-10</param>
+            <param name="max">10</param>
+        </command_interface>
+        <state_interface name="velocity"/>
+        <state_interface name="position"/>
+    </joint>
+    <joint name="right_wheel_joint">
+        <command_interface name="velocity">
+            <param name="min">-10</param>
+            <param name="max">10</param>
+        </command_interface>
+        <state_interface name="velocity"/>
+        <state_interface name="position"/>
+    </joint>
 </ros2_control>
 <gazebo>
